Commit message: updates

File: odrive_jeeves_description/urdf/odrive_jeeves.urdf.xacro (robot description, xacro)
@@ -10,5 +10,47 @@
     name="ODriveDiffBot"
     serial_number="2054368F424D"
-    joint0_name="$(arg prefix)Left_wheel_joint"
-    joint1_name="$(arg prefix)Right_wheel_joint" />
+    joint0_name="$(arg prefix)Right_wheel_joint"
+    joint1_name="$(arg prefix)Left_wheel_joint" />
+<!--
+// Copyright 2022 Stereolabs
+//
+// Licensed under the Apache License, Version 2.0 (the "License");
+// you may not use this file except in compliance with the License.
+// You may obtain a copy of the License at
+//
+//      http://www.apache.org/licenses/LICENSE-2.0
+//
+// Unless required by applicable law or agreed to in writing, software
+// distributed under the License is distributed on an "AS IS" BASIS,
+// WITHOUT WARRANTIES OR CONDITIONS OF ANY KIND, either express or implied.
+// See the License for the specific language governing permissions and
+// limitations under the License.
+-->
+  <xacro:arg name="camera_name"   default="zedm" />
+  <xacro:arg name="camera_model"  default="zedm" />
+  <xacro:arg name="base_frame"    default="Camera_IMU_1" />
+  <xacro:arg name="cam_pos_x"     default="0.0" />
+  <xacro:arg name="cam_pos_y"     default="0.0" />
+  <xacro:arg name="cam_pos_z"     default="0.0" />
+  <xacro:arg name="cam_roll"      default="0.0" />
+  <xacro:arg name="cam_pitch"     default="0.0" />
+  <xacro:arg name="cam_yaw"       default="0.0" />
+  <xacro:arg name="gnss_frame"    default="" />
+  <xacro:include filename="$(find zed_wrapper)/urdf/zed_macro.urdf.xacro" />
+  <xacro:zed_camera name="$(arg camera_name)" model="$(arg camera_model)" parent="$(arg base_frame)">
+    <origin
+      xyz="$(arg cam_pos_x) $(arg cam_pos_y) $(arg cam_pos_z)"
+      rpy="$(arg cam_roll) $(arg cam_pitch) $(arg cam_yaw)"
+    />
+  </xacro:zed_camera>
+  <xacro:property name="gnss_frame" value="$(arg gnss_frame)"/>
+  <!-- Set the position of the GNSS sensor relative to base_link if used -->
+  <xacro:if value="${gnss_frame != ''}">
+    <link name="$(arg gnss_frame)" />
+    <joint name="$(arg gnss_frame)_joint" type="fixed">
+      <parent link="$(arg base_frame)"/>
+      <child link="$(arg gnss_frame)"/>
+      <origin xyz="0 0 0.5" rpy="0 0 0" />
+    </joint>
+  </xacro:if>
 </robot>

Commit message: added realsense and top bottom camera

File: odrive_jeeves_description/urdf/odrive_jeeves.urdf.xacro (robot description, xacro)
@@ -15,5 +15,15 @@
     joint1_name="$(arg prefix)Right_wheel_joint"
     joint0_name="$(arg prefix)Left_wheel_joint" />
-<!--
+  <!--
+  <xacro:arg name="use_nominal_extrinsics" default="true"/>
+  <xacro:arg name="use_mesh" default="false"/>
+  <xacro:include filename="$(find realsense2_description)/urdf/_d435.urdf.xacro" />
+  <xacro:sensor_d435 parent="Camera_Top_1" name="rs_top" use_nominal_extrinsics="$(arg use_nominal_extrinsics)" use_mesh="$(arg use_mesh)">
+    <origin xyz="0 0 0" rpy="0 0.349066 0"/>
+  </xacro:sensor_d435>
+  <xacro:sensor_d435 parent="Camera_Bottom_1" name="rs_bottom" use_nominal_extrinsics="$(arg use_nominal_extrinsics)" use_mesh="$(arg use_mesh)">
+    <origin xyz="0 0 0" rpy="0 0 0" />
+  </xacro:sensor_d435>
+  -->
 // Copyright 2022 Stereolabs
 //
@@ -29,8 +39,7 @@
 // See the License for the specific language governing permissions and
 // limitations under the License.
--->
   <xacro:arg name="camera_name"   default="zedm" />
   <xacro:arg name="camera_model"  default="zedm" />
-  <xacro:arg name="base_frame"    default="Camera_IMU_Front_1" />
+  <xacro:arg name="base_frame"    default="Camera_Top_1" />
   <xacro:arg name="cam_pos_x"     default="0.0" />
   <xacro:arg name="cam_pos_y"     default="0.0" />
@@ -41,17 +50,17 @@
   <xacro:arg name="gnss_frame"    default="" />
   <xacro:include filename="$(find zed_wrapper)/urdf/zed_macro.urdf.xacro" />
-  <xacro:zed_camera name="zedm_front" model="$(arg camera_model)">
+  <xacro:zed_camera name="zedm_top" model="$(arg camera_model)">
   </xacro:zed_camera>
-  <joint name="Camera_IMU_Front_joint_f" type="fixed">
-    <origin xyz="0 0 0" rpy="0 -0.20943951023932 0"/>
-    <child link="zedm_front_camera_link"/>
-    <parent link="Camera_IMU_Front_1"/>
+  <joint name="Camera_IMU_Top_joint_f" type="fixed">
+    <origin xyz="0 0 0" rpy="0 0.349066 0"/>
+    <child link="zedm_top_camera_link"/>
+    <parent link="Camera_Top_1"/>
   </joint>
-  <xacro:zed_camera name="zedm_back" model="$(arg camera_model)">
+  <xacro:zed_camera name="zedm_bottom" model="$(arg camera_model)">
   </xacro:zed_camera>
-  <joint name="Camera_IMU_Back_joint_f" type="fixed">
-    <origin xyz="0 0 0" rpy="0 -0.20943951023932 3.141592653589793"/>
-    <child link="zedm_back_camera_link"/>
-    <parent link="Camera_IMU_Back_1"/>
+  <joint name="Camera_Bottom_joint_f" type="fixed">
+    <origin xyz="0 0 0" rpy="0 -0.436332 0"/>
+    <child link="zedm_bottom_camera_link"/>
+    <parent link="Camera_Bottom_1"/>
   </joint>
 </robot>
