Commit message: can drive working

File: odrive_jeeves_description/urdf/odrive.ros2_control.xacro (robot description, xacro)
@@ -2,5 +2,5 @@
 <robot xmlns:xacro="http://www.ros.org/wiki/xacro">
   <xacro:macro name="odrive_ros2_control"
-    params="name serial_number:=^|000000000000 enable_joint0:=^|true enable_joint1:=^|true joint0_name:=^|joint0 joint1_name:=^|joint1 can_tty:=^|can_tty can_speed:=^250000 joint0_canid:=^|1 joint1_canid:=^|2">
+    params="name serial_number:=^|000000000000 enable_joint0:=^|true enable_joint1:=^|true joint0_name:=^|joint0 joint1_name:=^|joint1 can_tty:=^|can_tty can_speed:=^250000 axis0_canid:=^|1 axis1_canid:=^|2">
     <ros2_control name="${name}" type="system">
       <hardware>
@@ -15,8 +15,8 @@
         <joint name="${joint0_name}">
           <param name="serial_number">${serial_number}</param>
-          <param name="axis">0</param>
-          <param name="can_id">${joint0_canid}</param>
+          <param name="axis">1</param>
+          <param name="can_id">${axis1_canid}</param>
           <param name="enable_watchdog">0</param>
-          <param name="reverse_control">0</param>
+          <param name="reverse_control">1</param>
           <param name="watchdog_timeout">0.1</param>
         </joint>
@@ -25,8 +25,8 @@
         <joint name="${joint1_name}">
           <param name="serial_number">${serial_number}</param>
-          <param name="axis">1</param>
-          <param name="can_id">${joint1_canid}</param>
+          <param name="axis">0</param>
+          <param name="can_id">${axis0_canid}</param>
           <param name="enable_watchdog">0</param>
-          <param name="reverse_control">1</param>
+          <param name="reverse_control">0</param>
           <param name="watchdog_timeout">0.1</param>
         </joint>

File: odrive_jeeves_description/urdf/odrive_jeeves.urdf.xacro (robot description, xacro)
@@ -11,6 +11,6 @@
     serial_number="2054368F424D"
     can_tty="/dev/ttyUSB0"
-    joint0_canid="1"
-    joint1_canid="2"
+    axis0_canid="1"
+    axis1_canid="2"
     joint1_name="$(arg prefix)Right_wheel_joint"
     joint0_name="$(arg prefix)Left_wheel_joint" />
@@ -32,5 +32,5 @@
   <xacro:arg name="camera_name"   default="zedm" />
   <xacro:arg name="camera_model"  default="zedm" />
-  <xacro:arg name="base_frame"    default="Camera_IMU_1" />
+  <xacro:arg name="base_frame"    default="Camera_IMU_Front_1" />
   <xacro:arg name="cam_pos_x"     default="0.0" />
   <xacro:arg name="cam_pos_y"     default="0.0" />
@@ -41,19 +41,17 @@
   <xacro:arg name="gnss_frame"    default="" />
   <xacro:include filename="$(find zed_wrapper)/urdf/zed_macro.urdf.xacro" />
-  <xacro:zed_camera name="$(arg camera_name)" model="$(arg camera_model)" parent="$(arg base_frame)">
-    <origin
-      xyz="$(arg cam_pos_x) $(arg cam_pos_y) $(arg cam_pos_z)"
-      rpy="$(arg cam_roll) $(arg cam_pitch) $(arg cam_yaw)"
-    />
+  <xacro:zed_camera name="zedm_front" model="$(arg camera_model)">
   </xacro:zed_camera>
-  <xacro:property name="gnss_frame" value="$(arg gnss_frame)"/>
-  <!-- Set the position of the GNSS sensor relative to base_link if used -->
-  <xacro:if value="${gnss_frame != ''}">
-    <link name="$(arg gnss_frame)" />
-    <joint name="$(arg gnss_frame)_joint" type="fixed">
-      <parent link="$(arg base_frame)"/>
-      <child link="$(arg gnss_frame)"/>
-      <origin xyz="0 0 0.5" rpy="0 0 0" />
-    </joint>
-  </xacro:if>
+  <joint name="Camera_IMU_Front_joint_f" type="fixed">
+    <origin xyz="0 0 0" rpy="0 -0.20943951023932 0"/>
+    <child link="zedm_front_camera_link"/>
+    <parent link="Camera_IMU_Front_1"/>
+  </joint>
+  <xacro:zed_camera name="zedm_back" model="$(arg camera_model)">
+  </xacro:zed_camera>
+  <joint name="Camera_IMU_Back_joint_f" type="fixed">
+    <origin xyz="0 0 0" rpy="0 -0.20943951023932 3.141592653589793"/>
+    <child link="zedm_back_camera_link"/>
+    <parent link="Camera_IMU_Back_1"/>
+  </joint>
 </robot>

Commit message: added many features

File: odrive_jeeves_description/urdf/odrive.ros2_control.xacro (robot description, xacro)
@@ -20,4 +20,6 @@
           <param name="reverse_control">1</param>
           <param name="watchdog_timeout">0.1</param>
+          <param name="vel_gain">4.361928939819336</param>
+          <param name="vel_integrator_gain">1.3249359130859375</param>
         </joint>
       </xacro:if>
@@ -30,4 +32,6 @@
           <param name="reverse_control">0</param>
           <param name="watchdog_timeout">0.1</param>
+          <param name="vel_gain">2.907952626546224</param>
+          <param name="vel_integrator_gain">1.3249359130859375</param>
         </joint>
       </xacro:if>

File: odrive_jeeves_description/urdf/odrive_jeeves.urdf.xacro (robot description, xacro)
@@ -15,15 +15,13 @@
     joint1_name="$(arg prefix)Right_wheel_joint"
     joint0_name="$(arg prefix)Left_wheel_joint" />
-  <!--
   <xacro:arg name="use_nominal_extrinsics" default="true"/>
   <xacro:arg name="use_mesh" default="false"/>
   <xacro:include filename="$(find realsense2_description)/urdf/_d435.urdf.xacro" />
   <xacro:sensor_d435 parent="Camera_Top_1" name="rs_top" use_nominal_extrinsics="$(arg use_nominal_extrinsics)" use_mesh="$(arg use_mesh)">
-    <origin xyz="0 0 0" rpy="0 0.349066 0"/>
+    <origin xyz="0 0 0" rpy="0 0 0"/>
   </xacro:sensor_d435>
   <xacro:sensor_d435 parent="Camera_Bottom_1" name="rs_bottom" use_nominal_extrinsics="$(arg use_nominal_extrinsics)" use_mesh="$(arg use_mesh)">
-    <origin xyz="0 0 0" rpy="0 0 0" />
+    <origin xyz="0 0 0" rpy="0 -0.436332  0" />
   </xacro:sensor_d435>
-  -->
 // Copyright 2022 Stereolabs
 //
@@ -39,4 +37,5 @@
 // See the License for the specific language governing permissions and
 // limitations under the License.
+<!--
   <xacro:arg name="camera_name"   default="zedm" />
   <xacro:arg name="camera_model"  default="zedm" />
@@ -53,5 +52,5 @@
   </xacro:zed_camera>
   <joint name="Camera_IMU_Top_joint_f" type="fixed">
-    <origin xyz="0 0 0" rpy="0 0.349066 0"/>
+    <origin xyz="0 0 0" rpy="0 0 0"/>
     <child link="zedm_top_camera_link"/>
     <parent link="Camera_Top_1"/>
@@ -64,3 +63,4 @@
     <parent link="Camera_Bottom_1"/>
   </joint>
+-->
 </robot>
